Commit message: update to governatorusv

File: governatorusv_description/urdf/snippets.xacro (robot description, xacro)
@@ -5,5 +5,5 @@
   over propeller's frame X-axis in DAE (Collada) or STL format.
   -->
-  <xacro:property name="prop_mesh_file" value="file://$(find minionusv_description)/meshes/propeller.dae"/>
+  <xacro:property name="prop_mesh_file" value="file://$(find governator_description)/meshes/propeller.dae"/>
   <!--
     Thruster macro with integration of joint and link. The thrusters should
