Commit message: update to governatorsuv

File: governatorusv_description/robots/governator_default.xacro (robot description, xacro)
@@ -1,11 +1,11 @@
 <?xml version="1.0"?>
-<robot name="governatorusv" xmlns:xacro="http://www.ros.org/wiki/xacro" >
+<robot name="governator" xmlns:xacro="http://www.ros.org/wiki/xacro" >
   <xacro:arg name="debug" default="0"/>
-  <xacro:arg name="namespace" default="governatorusv"/>
+  <xacro:arg name="namespace" default="governator"/>
   <!-- Include the ROV macro file -->
-  <xacro:include filename="$(find governatorusv_description)/urdf/base.xacro"/>
-  <xacro:include filename="$(find governatorusv_description)/urdf/gazebo.xacro"/>
-  <!-- Create the governatorusv -->
-  <xacro:governatorusv_base namespace="$(arg namespace)">
+  <xacro:include filename="$(find governator_description)/urdf/base.xacro"/>
+  <xacro:include filename="$(find governator_description)/urdf/gazebo.xacro"/>
+<!-- Create the governator -->
+  <xacro:governator_base namespace="$(arg namespace)">
     <!-- The underwater object plugin is given as an input block parameter to
      allow the addition of external models of manipulator units -->
@@ -15,6 +15,6 @@
         <flow_velocity_topic>hydrodynamics/current_velocity</flow_velocity_topic>
         <debug>$(arg debug)</debug>
-        <!-- Adding the hydrodynamic and hydrostatic parameters for the vehicle-->
-        <xacro:governatorusv_hydro_model namespace="$(arg namespace)"/>
+        <!-- Adding the hydrodynamic and hydrostatic parameters for the vehicle -->
+        <xacro:governator_hydro_model namespace="$(arg namespace)"/>
         <!--
           In case other modules are added to the vehicle (such as a manipulator)
@@ -26,5 +26,5 @@
       </plugin>
     </gazebo>
-  </xacro:governatorusv_base>
+  </xacro:governator_base>
   <!-- Joint state publisher plugin -->
   <xacro:default_joint_state_publisher namespace="$(arg namespace)" update_rate="50"/>

File: governatorusv_description/urdf/base.xacro (robot description, xacro)
@@ -6,9 +6,12 @@
   <xacro:include filename="$(find uuv_sensor_ros_plugins)/urdf/sensor_snippets.xacro"/>
   <!-- Loading vehicle's specific macros -->
-  <xacro:include filename="$(find governatorusv_description)/urdf/snippets.xacro"/>
+  <xacro:include filename="$(find governator_description)/urdf/snippets.xacro"/>
+  <!-- ADDED  -->
+  <xacro:include filename="$(find uuv_gazebo_ros_plugins)/urdf/snippets.xacro"/>
   <!--
     Vehicle's parameters (remember to enter the model parameters below)
   -->
-  <xacro:property name="mass" value="0"/>
+  <!-- Mass, see p.28 in Berg2012 -->
+  <xacro:property name="mass" value="1862.87"/>
   <!-- Center of gravity -->
   <xacro:property name="cog" value="0 0 0"/>
@@ -21,11 +24,12 @@
     Open the meshes for the RexROV vehicle in Blender to see an example on the mesh placement.
   -->
-  <xacro:property name="visual_mesh_file" value="file://$(find governatorusv_description)/meshes/vehicle.dae"/>
+  <xacro:property name="visual_mesh_file" value="file://$(find governator_description)/meshes/governator.dae"/>
   <!-- Collision geometry mesh, usually in STL format (it is recommended to keep
   this geometry as simple as possible to improve the performance the physics engine
   regarding the computation of collision forces) -->
-  <xacro:property name="collision_mesh_file" value="file://$(find governatorusv_description)/meshes/vehicle.stl"/>
+  <xacro:property name="collision_mesh_file" value="file://$(find governator_description)/meshes/governator.stl"/>
   <!-- Vehicle macro -->
-  <xacro:macro name="governatorusv_base" params="namespace debug *gazebo">
+  <!-- <xacro:macro name="governator_base" params="namespace debug *gazebo"> -->
+  <xacro:macro name="governator_base" params="namespace *gazebo">
       <!-- Rigid body description of the base link -->
       <link name="${namespace}/base_link">
@@ -37,8 +41,11 @@
           <mass value="${mass}" />
           <origin xyz="${cog}" rpy="0 0 0"/>
-          <inertia ixx="0" ixy="0" ixz="0"
-                   iyy="0" iyz="0"
-                   izz="0" />
+          <inertia ixx="525.39" ixy="1.44" ixz="33.41" iyy="794.20" iyz="2.6" izz="691.23"/>
         </inertial>
+        <!-- This visual geometry representation can be used when running
+             tasks in which you need Gazebo to start quickly
+        -->
+        <!-- <xacro:if value="${use_simplified_mesh}"> -->
+        <!-- Code in rexrov2_base.xacro if use the flag use_simplified_mesh -->
         <visual>
           <origin xyz="0 0 0" rpy="0 0 0"/>
@@ -47,4 +54,5 @@
           </geometry>
         </visual>
+        <!-- In rexrov2_base they made collision planes -->
         <collision>
           <origin xyz="0 0 0" rpy="0 0 0"/>
@@ -54,13 +62,14 @@
         </collision>
       </link>
-    <gazebo reference="${namespace}/base_link">
+    <!-- <gazebo reference="${namespace}/base_link">
       <selfCollide>false</selfCollide>
-    </gazebo>
+    </gazebo> -->
     <!-- Set up hydrodynamic plugin given as input parameter -->
     <xacro:insert_block name="gazebo"/>
+    <!-- !!!!!!TO DO LATER!!!!! -->
     <!-- Include the thruster modules -->
-    <xacro:include filename="$(find governatorusv_description)/urdf/thrusters.xacro"/>
+    <!-- <xacro:include filename="$(find governator_description)/urdf/thrusters.xacro"/> -->
     <!-- Include the sensor modules -->
-    <xacro:include filename="$(find governatorusv_description)/urdf/sensors.xacro"/>
+    <!-- <xacro:include filename="$(find governator_description)/urdf/sensors.xacro"/> -->
   </xacro:macro>
 </robot>

File: governatorusv_description/urdf/gazebo.xacro (robot description, xacro)
@@ -1,56 +1,56 @@
 <?xml version="1.0"?>
 <robot xmlns:xacro="http://www.ros.org/wiki/xacro">
-    <!-- Center of buoyancy -->
-    <xacro:property name="governatorusv_cob" value="0 0 0"/>
-    <!-- Vehicle's actual volume (Gazebo cannot compute the volume out of the mesh) -->
-    <xacro:property name="governatorusv_volume" value="0"/>
-    <!-- Describing the dimensions of the vehicle's bounding box -->
-    <xacro:property name="governatorusv_length" value="0"/>
-    <xacro:property name="governatorusv_width"  value="0"/>
-    <xacro:property name="governatorusv_height" value="0"/>
-    <xacro:macro name="governatorusv_hydro_model" params="namespace">
-      <!-- List of hydrodynamic models this robot's links -->
-      <link name="${namespace}/base_link">
-        <!-- This flag will make the link neutrally buoyant -->
-        <neutrally_buoyant>0</neutrally_buoyant>
-        <!-- Link's volume -->
-        <volume>${governatorusv_volume}</volume>
-        <!-- Link's bounding box, it is used to recalculate the immersed
+  <!--
+  Center of buoyancy according to eq. (3.1) p. 28 in Berg2012.
+  The original values, [0.0822, -0.00773, 0.3872] however, seem to
+  assume NWU (otherwise cob is below cog?).
+  -->
+  <xacro:property name="governator_cob" value="0.0 0.0 0.3"/>
+  <!-- Volume, see p.31 in Berg2012 -->
+  <xacro:property name="governator_volume" value="1.83826"/>
+  <!-- Describing the dimensions of the vehicle's bounding box -->
+  <xacro:property name="governator_length" value="1"/>
+  <xacro:property name="governator_width"  value="1"/>
+  <xacro:property name="governator_height" value="1"/>
+  <xacro:macro name="governator_hydro_model" params="namespace">
+    <!-- List of hydrodynamic models this robot's links -->
+    <link name="${namespace}/base_link">
+      <!-- This flag will make the link neutrally buoyant -->
+      <neutrally_buoyant>0</neutrally_buoyant>
+      <!-- Link's volume -->
+      <volume>${governator_volume}</volume>
+      <!-- Link's bounding box, it is used to recalculate the immersed
         volume when close to the surface.
         This is a workaround the invalid bounding box given by Gazebo-->
-        <box>
-          <width>${governatorusv_width}</width>
-          <length>${governatorusv_length}</length>
-          <height>${governatorusv_height}</height>
-        </box>
-        <!-- Center of buoyancy -->
-        <center_of_buoyancy>${governatorusv_cob}</center_of_buoyancy>
-        <!--
-        ----------------------------------------------------
-        ----------------------------------------------------
-        Choose one of the hydrodynamic models below, all are based on
-        Fossen's equation of motion for underwater vehicles
-        Reference:
-        [1] Fossen, Thor I. Handbook of marine craft hydrodynamics and motion
-            control. John Wiley & Sons, 2011.
-        ----------------------------------------------------
-        ---------------------------------------------------->
-        <!-- 1) Fossen's equation of motion -->
-        <hydrodynamic_model>
+      <box>
+        <width>${governator_width}</width>
+        <length>${governator_length}</length>
+        <height>${governator_height}</height>
+      </box>
+      <!-- Center of buoyancy -->
+      <center_of_buoyancy>${governator_cob}</center_of_buoyancy>
+      <!-- Fossen's equation of motion for underwater vehicles
+      Reference:
+          [1] Fossen, Thor I. Handbook of marine craft hydrodynamics and motion
+          control. John Wiley & Sons, 2011.
+     -->
+      <hydrodynamic_model>
           <type>fossen</type>
+          <!-- Added mass: see p.28 in Berg2012 -->
           <added_mass>
-            0 0 0 0 0 0
-            0 0 0 0 0 0
-            0 0 0 0 0 0
-            0 0 0 0 0 0
-            0 0 0 0 0 0
-            0 0 0 0 0 0
+            779.79 -6.8773 -103.32  8.5426 -165.54 -7.8033
+           -6.8773    1222   51.29  409.44 -5.8488  62.726
+           -103.32   51.29  3659.9  6.1112 -386.42  10.774
+            8.5426  409.44  6.1112   534.9 -10.027  21.019
+           -165.54 -5.8488 -386.42 -10.027  842.69 -1.1162
+           -7.8033  62.726  10.775  21.019 -1.1162  224.32
           </added_mass>
           <!--
             The linear damping coefficients can be provided as a diagonal (6 elements)
             or a full matrix (36 coefficients), like the added-mass coefficients above
+            Linear damping: see p.31 in Berg2012
           -->
           <linear_damping>
-            0 0 0 0 0 0
+            -74.82 -69.48 -728.4 -268.8 -309.77 -105
           </linear_damping>
           <!--
@@ -60,13 +60,14 @@
             This matrix is mostly useful for slender bodies (e.g. AUVs with torpedo shape)
           -->
-          <linear_damping_forward_speed>
+          <!-- <linear_damping_forward_speed>
             0 0 0 0 0 0
-          </linear_damping_forward_speed>
+          </linear_damping_forward_speed> -->
           <!--
             The quadratic damping coefficients can be provided as a diagonal (6 elements)
             or a full matrix (36 coefficients), like the added-mass coefficients above
+            Non-linear damping: see p.30 in Berg2012
           -->
           <quadratic_damping>
-            0 0 0 0 0 0
+            -748.22 -992.53 -1821.01 -672 -774.44 -523.27
           </quadratic_damping>
           <!--
@@ -84,17 +85,9 @@
                   control. John Wiley & Sons, 2011.
           -->
-          <!--
-          <metacentric_width>0.0</metacentric_width>
-          <metacentric_length>0.0</metacentric_length>
-          <water_level_plane_area>0.0</water_level_plane_area>
-          -->
-        </hydrodynamic_model>
-        <!-- 2) This computes the added-mass and damping parameters for a sphere
-        in the fluid with the given radius -->
-        <hydrodynamic_model>
-          <type>sphere</type>
-          <radius>0</radius>
-        </hydrodynamic_model>
-      </link>
-    </xacro:macro>
+          <metacentric_width>0.2</metacentric_width>
+          <metacentric_length>0.2</metacentric_length>
+          <water_level_plane_area>0.04</water_level_plane_area>
+      </hydrodynamic_model>
+    </link>
+  </xacro:macro>
 </robot>

File: governatorusv_description/urdf/snippets.xacro (robot description, xacro)
@@ -1,11 +1,9 @@
 <?xml version="1.0"?>
 <robot xmlns:xacro="http://www.ros.org/wiki/xacro">
-  <!-------------------------------------------------------------------------->
   <!-- MACRO FOR THRUSTER UNITS  -->
-  <!-------------------------------------------------------------------------->
   <!-- Provide the propeller mesh in a separate file with the rotation axis
   over propeller's frame X-axis in DAE (Collada) or STL format.
   -->
-  <xacro:property name="prop_mesh_file" value="file://$(find governatorusv_description)/meshes/propeller.dae"/>
+  <xacro:property name="prop_mesh_file" value="file://$(find minionusv_description)/meshes/propeller.dae"/>
   <!--
     Thruster macro with integration of joint and link. The thrusters should
@@ -70,11 +68,7 @@
         <propeller_efficiency>1</propeller_efficiency>
         <!--
-        ----------------------------------------------------
-        ----------------------------------------------------
         Choose one of the propeller dynamics models below for your implementation
         This will describe the dynamic model for the state variable of your thruster unit,
-        which can be, e.g., the angular velocity of the propeller.
-        ----------------------------------------------------
-        ---------------------------------------------------->
+        which can be, e.g., the angular velocity of the propeller. -->
         <!-- 1) Simple zero-order model -->
         <dynamics>
@@ -82,8 +76,8 @@
         </dynamics>
         <!-- 2) First order model -->
-        <dynamics>
+        <!-- <dynamics>
           <type>FirstOrder</type>
           <timeConstant>0.0</timeConstant>
-        </dynamics>
+        </dynamics> -->
         <!-- 3) Yoerger's nonlinear dynamic model
         For information on the model description:
@@ -93,9 +87,9 @@
             no. 3, pp. 167–178, Jul. 1990.
         -->
-        <dynamics>
+        <!-- <dynamics>
           <type>Yoerger</type>
           <alpha>0.0</alpha>
           <beta>0.0</beta>
-        </dynamics>
+        </dynamics> -->
         <!-- 4) Bessa's nonlinear dynamic model
         For information on the model description:
@@ -105,5 +99,5 @@
             Mechatronics. Vol. 2. 2006.
         -->
-        <dynamics>
+        <!-- <dynamics>
           <type>Bessa</type>
           <Jmsp>0.0</Jmsp>
@@ -112,12 +106,8 @@
           <Kt>0.0</Kt>
           <Rm>0.0</Rm>
-        </dynamics>
+        </dynamics> -->
         <!--
-        ----------------------------------------------------
-        ----------------------------------------------------
         Choose one of the model for the steady-state curve describing the
-        relationship between the state variable and the output thrust force
-        ----------------------------------------------------
-        ---------------------------------------------------->
+        relationship between the state variable and the output thrust force -->
         <!-- 1) Basic curve
         Input: x
@@ -137,5 +127,5 @@
         thrust = rotorConstantR * (x * abs(x) - deltaR), if x * abs(x) >= deltaL
         -->
-        <conversion>
+        <!-- <conversion>
           <type>Bessa</type>
           <rotorConstantL>0.0</rotorConstantL>
@@ -143,5 +133,5 @@
           <deltaL>0.0</deltaL>
           <deltaR>0.0</deltaR>
-        </conversion>
+        </conversion> -->
         <!-- 3) Linear interpolation
         If you have access to the thruster's data sheet, for example,
@@ -150,118 +140,14 @@
         of the given samples.
         -->
-        <conversion>
+        <!-- <conversion>
           <type>LinearInterp</type>
           <inputValues>0 1 2 3</inputValues>
           <outputValues>0 1 2 3</outputValues>
-        </conversion>
+        </conversion> -->
       </plugin>
     </gazebo>
-    <gazebo reference="${robot_namespace}/thruster_${thruster_id}">
+    <!-- <gazebo reference="${robot_namespace}/thruster_${thruster_id}">
       <selfCollide>false</selfCollide>
-    </gazebo>
-  </xacro:macro>
-  <!-------------------------------------------------------------------------->
-  <!-- MACRO FOR FIN/RUDDER UNITS  -->
-  <!-------------------------------------------------------------------------->
-  <!--
-    This macro can be used to add fins to the body of the vehicle, the fins
-    should be initialized in the actuators.xacro file. If you vehicle has no
-    fins, you can erase the macro below.
-  -->
-  <!-- A separate mesh for the fin should be stored in the meshes folder -->
-  <xacro:property name="fin_mesh_file" value="file://$(find governatorusv_description)/meshes/fin.dae"/>
-  <!-- Fin joint limits  -->
-  <xacro:property name="fin_min_joint_limit" value="${0.0 * d2r}"/>
-  <xacro:property name="fin_max_joint_limit" value="${0.0 * d2r}"/>
-  <xacro:macro name="fin_macro" params="namespace fin_id *origin">
-      <joint name="${namespace}/fin${fin_id}_joint" type="revolute">
-          <limit effort="0" lower="${fin_min_joint_limit}" upper="${fin_max_joint_limit}" velocity="0"/>
-          <xacro:insert_block name="origin"/>
-          <axis xyz="0 0 1"/>
-          <parent link="${namespace}/base_link" />
-          <child link="${namespace}/fin${fin_id}" />
-      </joint>
-      <link name="${namespace}/fin${fin_id}">
-        <inertial>
-          <mass value="0.001" />
-          <origin xyz="0 0 0" rpy="0 0 0"/>
-          <inertia ixx="0.000000017" ixy="0.0" ixz="0.0"
-                 iyy="0.000000017" iyz="0.0"
-                 izz="0.000000017" />
-        </inertial>
-        <visual>
-          <origin xyz="0 0 0" rpy="0 0 0" />
-          <geometry>
-            <mesh filename="${fin_mesh_file}" scale="1 1 1"/>
-          </geometry>
-        </visual>
-      </link>
-      <gazebo>
-        <plugin name="${namespace}_fin${fin_id}_model" filename="libfin_ros_plugin.so">
-          <!--
-            ----------------------------------------------------
-            ----------------------------------------------------
-            First order dynamics model for the fin joint dynamics,
-            replace an appropriate time constant
-            ----------------------------------------------------
-            ----------------------------------------------------
-          -->
-          <dynamics>
-            <type>FirstOrder</type>
-            <timeConstant>0.0</timeConstant>
-          </dynamics>
-          <!--
-            ----------------------------------------------------
-            ----------------------------------------------------
-            Definition of the lift and drag model, choose ONE of the models
-            below according to the model you want to use.
-            ----------------------------------------------------
-            ----------------------------------------------------
-          -->
-          <!--
-            1) References for the two line lift and drag model:
-              [1] https://en.wikipedia.org/wiki/Lift_coefficient
-              [2] http://gazebosim.org/tutorials?tut=aerodynamics&cat=plugins
-          -->
-          <liftdrag>
-            <type>TwoLines</type>
-            <area>${replace here the value for the area of the fin's cross section}</area>
-            <fluid_density>0.0</fluid_density>
-            <a0>0.0</a0>
-            <alpha_stall>0.0</alpha_stall>
-            <cla>0.0</cla><!-- ^= 0.244 when using deg -->
-            <cla_stall>0.0</cla_stall>
-            <cda>0.0</cda>
-            <cda_stall>0.0</cda_stall>
-          </liftdrag>
-          <!--
-            2) Reference for the quadratic lift and drag model:
-              [1] Engelhardtsen, Oystein. 3D AUV Collision Avoidance.
-                  MS thesis. Institutt for teknisk kybernetikk, 2007.
-                  https://brage.bibsys.no/xmlui/handle/11250/259834
-          -->
-          <liftdrag>
-            <type>Quadratic</type>
-            <lift_constant>0.0</lift_constant>
-            <drag_constant>0.0</drag_constant>
-          </liftdrag>
-          <!--
-            ----------------------------------------------------
-            ----------------------------------------------------
-            Further parameters necessary for the lift and drag plugin
-            ----------------------------------------------------
-            ----------------------------------------------------
-          -->
-          <!-- Current velocity topic -->
-          <current_velocity_topic>/hydrodynamics/current_velocity</current_velocity_topic>
-          <!-- Name of the correspodent fin link and joint  -->
-          <link_name>${namespace}/fin${fin_id}</link_name>
-          <joint_name>${namespace}/fin${fin_id}_joint</joint_name>
-          <!-- Output topic to publish the current angle of the fin joint -->
-          <output_topic>${namespace}/fins/${fin_id}/output</output_topic>
-          <input_topic>${namespace}/fins/${fin_id}/input</input_topic>
-          <wrench_topic>${namespace}/fins/${fin_id}/wrench_topic</wrench_topic>
-        </plugin>
-      </gazebo>
+    </gazebo> -->
   </xacro:macro>
 </robot>
