Commit message: change to governatorusv, correct the error

File: governatorusv_description/robots/governator_default.xacro (robot description, xacro)
@@ -1,11 +1,11 @@
 <?xml version="1.0"?>
-<robot name="governator" xmlns:xacro="http://www.ros.org/wiki/xacro" >
+<robot name="governatorusv" xmlns:xacro="http://www.ros.org/wiki/xacro" >
   <xacro:arg name="debug" default="0"/>
-  <xacro:arg name="namespace" default="governator"/>
+  <xacro:arg name="namespace" default="governatorusv"/>
   <!-- Include the ROV macro file -->
-  <xacro:include filename="$(find governator_description)/urdf/base.xacro"/>
-  <xacro:include filename="$(find governator_description)/urdf/gazebo.xacro"/>
-<!-- Create the governator -->
-  <xacro:governator_base namespace="$(arg namespace)">
+  <xacro:include filename="$(find governatorusv_description)/urdf/base.xacro"/>
+  <xacro:include filename="$(find governatorusv_description)/urdf/gazebo.xacro"/>
+<!-- Create the governatorusv -->
+  <xacro:governatorusv_base namespace="$(arg namespace)">
     <!-- The underwater object plugin is given as an input block parameter to
      allow the addition of external models of manipulator units -->
@@ -16,5 +16,5 @@
         <debug>$(arg debug)</debug>
         <!-- Adding the hydrodynamic and hydrostatic parameters for the vehicle -->
-        <xacro:governator_hydro_model namespace="$(arg namespace)"/>
+        <xacro:governatorusv_hydro_model namespace="$(arg namespace)"/>
         <!--
           In case other modules are added to the vehicle (such as a manipulator)
@@ -26,5 +26,5 @@
       </plugin>
     </gazebo>
-  </xacro:governator_base>
+  </xacro:governatorusv_base>
   <!-- Joint state publisher plugin -->
   <xacro:default_joint_state_publisher namespace="$(arg namespace)" update_rate="50"/>

File: governatorusv_description/urdf/base.xacro (robot description, xacro)
@@ -6,5 +6,5 @@
   <xacro:include filename="$(find uuv_sensor_ros_plugins)/urdf/sensor_snippets.xacro"/>
   <!-- Loading vehicle's specific macros -->
-  <xacro:include filename="$(find governator_description)/urdf/snippets.xacro"/>
+  <xacro:include filename="$(find governatorusv_description)/urdf/snippets.xacro"/>
   <!-- ADDED  -->
   <xacro:include filename="$(find uuv_gazebo_ros_plugins)/urdf/snippets.xacro"/>
@@ -24,12 +24,12 @@
     Open the meshes for the RexROV vehicle in Blender to see an example on the mesh placement.
   -->
-  <xacro:property name="visual_mesh_file" value="file://$(find governator_description)/meshes/governator.dae"/>
+  <xacro:property name="visual_mesh_file" value="file://$(find governatorusv_description)/meshes/governatorusv.dae"/>
   <!-- Collision geometry mesh, usually in STL format (it is recommended to keep
   this geometry as simple as possible to improve the performance the physics engine
   regarding the computation of collision forces) -->
-  <xacro:property name="collision_mesh_file" value="file://$(find governator_description)/meshes/governator.stl"/>
+  <xacro:property name="collision_mesh_file" value="file://$(find governatorusv_description)/meshes/governatorusv.stl"/>
   <!-- Vehicle macro -->
-  <!-- <xacro:macro name="governator_base" params="namespace debug *gazebo"> -->
-  <xacro:macro name="governator_base" params="namespace *gazebo">
+  <!-- <xacro:macro name="governatorusv_base" params="namespace debug *gazebo"> -->
+  <xacro:macro name="governatorusv_base" params="namespace *gazebo">
       <!-- Rigid body description of the base link -->
       <link name="${namespace}/base_link">
@@ -69,7 +69,7 @@
     <!-- !!!!!!TO DO LATER!!!!! -->
     <!-- Include the thruster modules -->
-    <!-- <xacro:include filename="$(find governator_description)/urdf/thrusters.xacro"/> -->
+    <!-- <xacro:include filename="$(find governatorusv_description)/urdf/thrusters.xacro"/> -->
     <!-- Include the sensor modules -->
-    <!-- <xacro:include filename="$(find governator_description)/urdf/sensors.xacro"/> -->
+    <!-- <xacro:include filename="$(find governatorusv_description)/urdf/sensors.xacro"/> -->
   </xacro:macro>
 </robot>

File: governatorusv_description/urdf/gazebo.xacro (robot description, xacro)
@@ -6,12 +6,12 @@
   assume NWU (otherwise cob is below cog?).
   -->
-  <xacro:property name="governator_cob" value="0.0 0.0 0.3"/>
+  <xacro:property name="governatorusv_cob" value="0.0 0.0 0.3"/>
   <!-- Volume, see p.31 in Berg2012 -->
-  <xacro:property name="governator_volume" value="1.83826"/>
+  <xacro:property name="governatorusv_volume" value="1.83826"/>
   <!-- Describing the dimensions of the vehicle's bounding box -->
-  <xacro:property name="governator_length" value="1"/>
-  <xacro:property name="governator_width"  value="1"/>
-  <xacro:property name="governator_height" value="1"/>
-  <xacro:macro name="governator_hydro_model" params="namespace">
+  <xacro:property name="governatorusv_length" value="1"/>
+  <xacro:property name="governatorusv_width"  value="1"/>
+  <xacro:property name="governatorusv_height" value="1"/>
+  <xacro:macro name="governatorusv_hydro_model" params="namespace">
     <!-- List of hydrodynamic models this robot's links -->
     <link name="${namespace}/base_link">
@@ -19,15 +19,15 @@
       <neutrally_buoyant>0</neutrally_buoyant>
       <!-- Link's volume -->
-      <volume>${governator_volume}</volume>
+      <volume>${governatorusv_volume}</volume>
       <!-- Link's bounding box, it is used to recalculate the immersed
         volume when close to the surface.
         This is a workaround the invalid bounding box given by Gazebo-->
       <box>
-        <width>${governator_width}</width>
-        <length>${governator_length}</length>
-        <height>${governator_height}</height>
+        <width>${governatorusv_width}</width>
+        <length>${governatorusv_length}</length>
+        <height>${governatorusv_height}</height>
       </box>
       <!-- Center of buoyancy -->
-      <center_of_buoyancy>${governator_cob}</center_of_buoyancy>
+      <center_of_buoyancy>${governatorusv_cob}</center_of_buoyancy>
       <!-- Fossen's equation of motion for underwater vehicles
       Reference:

File: governatorusv_description/urdf/snippets.xacro (robot description, xacro)
@@ -5,5 +5,5 @@
   over propeller's frame X-axis in DAE (Collada) or STL format.
   -->
-  <xacro:property name="prop_mesh_file" value="file://$(find governator_description)/meshes/propeller.dae"/>
+  <xacro:property name="prop_mesh_file" value="file://$(find governatorusv_description)/meshes/propeller.dae"/>
   <!--
     Thruster macro with integration of joint and link. The thrusters should
