Commit message: yet in renamed to ros convetion

File: governator_usv_description/robots/governator_usv_default.xacro (robot description, xacro)
@@ -1,11 +1,11 @@
 <?xml version="1.0"?>
-<robot name="governatorusv" xmlns:xacro="http://www.ros.org/wiki/xacro" >
+<robot name="governator_usv" xmlns:xacro="http://www.ros.org/wiki/xacro" >
   <xacro:arg name="debug" default="0"/>
-  <xacro:arg name="namespace" default="governatorusv"/>
+  <xacro:arg name="namespace" default="governator_usv"/>
   <!-- Include the ROV macro file -->
-  <xacro:include filename="$(find governatorusv_description)/urdf/base.xacro"/>
-  <xacro:include filename="$(find governatorusv_description)/urdf/gazebo.xacro"/>
-<!-- Create the governatorusv -->
-  <xacro:governatorusv_base namespace="$(arg namespace)">
+  <xacro:include filename="$(find governator_usv_description)/urdf/base.xacro"/>
+  <xacro:include filename="$(find governator_usv_description)/urdf/gazebo.xacro"/>
+<!-- Create the governator_usv -->
+  <xacro:governator_usv_base namespace="$(arg namespace)">
     <!-- The underwater object plugin is given as an input block parameter to
      allow the addition of external models of manipulator units -->
@@ -16,5 +16,5 @@
         <debug>$(arg debug)</debug>
         <!-- Adding the hydrodynamic and hydrostatic parameters for the vehicle -->
-        <xacro:governatorusv_hydro_model namespace="$(arg namespace)"/>
+        <xacro:governator_usv_hydro_model namespace="$(arg namespace)"/>
         <!--
           In case other modules are added to the vehicle (such as a manipulator)
@@ -26,5 +26,5 @@
       </plugin>
     </gazebo>
-  </xacro:governatorusv_base>
+  </xacro:governator_usv_base>
   <!-- Joint state publisher plugin -->
   <xacro:default_joint_state_publisher namespace="$(arg namespace)" update_rate="50"/>

File: governator_usv_description/urdf/base.xacro (robot description, xacro)
@@ -6,5 +6,5 @@
   <xacro:include filename="$(find uuv_sensor_ros_plugins)/urdf/sensor_snippets.xacro"/>
   <!-- Loading vehicle's specific macros -->
-  <xacro:include filename="$(find governatorusv_description)/urdf/snippets.xacro"/>
+  <xacro:include filename="$(find governator_usv_description)/urdf/snippets.xacro"/>
   <!-- ADDED  -->
   <xacro:include filename="$(find uuv_gazebo_ros_plugins)/urdf/snippets.xacro"/>
@@ -24,12 +24,12 @@
     Open the meshes for the RexROV vehicle in Blender to see an example on the mesh placement.
   -->
-  <xacro:property name="visual_mesh_file" value="file://$(find governatorusv_description)/meshes/governatorusv.dae"/>
+  <xacro:property name="visual_mesh_file" value="file://$(find governator_usv_description)/meshes/governator_usv.dae"/>
   <!-- Collision geometry mesh, usually in STL format (it is recommended to keep
   this geometry as simple as possible to improve the performance the physics engine
   regarding the computation of collision forces) -->
-  <xacro:property name="collision_mesh_file" value="file://$(find governatorusv_description)/meshes/governatorusv.stl"/>
+  <xacro:property name="collision_mesh_file" value="file://$(find governator_usv_description)/meshes/governator_usv.stl"/>
   <!-- Vehicle macro -->
-  <!-- <xacro:macro name="governatorusv_base" params="namespace debug *gazebo"> -->
-  <xacro:macro name="governatorusv_base" params="namespace *gazebo">
+  <!-- <xacro:macro name="governator_usv_base" params="namespace debug *gazebo"> -->
+  <xacro:macro name="governator_usv_base" params="namespace *gazebo">
       <!-- Rigid body description of the base link -->
       <link name="${namespace}/base_link">
@@ -69,7 +69,7 @@
     <!-- !!!!!!TO DO LATER!!!!! -->
     <!-- Include the thruster modules -->
-    <!-- <xacro:include filename="$(find governatorusv_description)/urdf/thrusters.xacro"/> -->
+    <!-- <xacro:include filename="$(find governator_usv_description)/urdf/thrusters.xacro"/> -->
     <!-- Include the sensor modules -->
-    <!-- <xacro:include filename="$(find governatorusv_description)/urdf/sensors.xacro"/> -->
+    <!-- <xacro:include filename="$(find governator_usv_description)/urdf/sensors.xacro"/> -->
   </xacro:macro>
 </robot>

File: governator_usv_description/urdf/gazebo.xacro (robot description, xacro)
@@ -6,12 +6,12 @@
   assume NWU (otherwise cob is below cog?).
   -->
-  <xacro:property name="governatorusv_cob" value="0.0 0.0 0.3"/>
+  <xacro:property name="governator_usv_cob" value="0.0 0.0 0.3"/>
   <!-- Volume, see p.31 in Berg2012 -->
-  <xacro:property name="governatorusv_volume" value="1.83826"/>
+  <xacro:property name="governator_usv_volume" value="1.83826"/>
   <!-- Describing the dimensions of the vehicle's bounding box -->
-  <xacro:property name="governatorusv_length" value="1"/>
-  <xacro:property name="governatorusv_width"  value="1"/>
-  <xacro:property name="governatorusv_height" value="1"/>
-  <xacro:macro name="governatorusv_hydro_model" params="namespace">
+  <xacro:property name="governator_usv_length" value="1"/>
+  <xacro:property name="governator_usv_width"  value="1"/>
+  <xacro:property name="governator_usv_height" value="1"/>
+  <xacro:macro name="governator_usv_hydro_model" params="namespace">
     <!-- List of hydrodynamic models this robot's links -->
     <link name="${namespace}/base_link">
@@ -19,15 +19,15 @@
       <neutrally_buoyant>0</neutrally_buoyant>
       <!-- Link's volume -->
-      <volume>${governatorusv_volume}</volume>
+      <volume>${governator_usv_volume}</volume>
       <!-- Link's bounding box, it is used to recalculate the immersed
         volume when close to the surface.
         This is a workaround the invalid bounding box given by Gazebo-->
       <box>
-        <width>${governatorusv_width}</width>
-        <length>${governatorusv_length}</length>
-        <height>${governatorusv_height}</height>
+        <width>${governator_usv_width}</width>
+        <length>${governator_usv_length}</length>
+        <height>${governator_usv_height}</height>
       </box>
       <!-- Center of buoyancy -->
-      <center_of_buoyancy>${governatorusv_cob}</center_of_buoyancy>
+      <center_of_buoyancy>${governator_usv_cob}</center_of_buoyancy>
       <!-- Fossen's equation of motion for underwater vehicles
       Reference:

File: governator_usv_description/urdf/snippets.xacro (robot description, xacro)
@@ -5,5 +5,5 @@
   over propeller's frame X-axis in DAE (Collada) or STL format.
   -->
-  <xacro:property name="prop_mesh_file" value="file://$(find governatorusv_description)/meshes/propeller.dae"/>
+  <xacro:property name="prop_mesh_file" value="file://$(find governator_usv_description)/meshes/propeller.dae"/>
   <!--
     Thruster macro with integration of joint and link. The thrusters should
